Commit message: add gripper

File: r12_description/urdf/r12.urdf (robot description, URDF)
Before this commit: robot r12, 6 links, 5 joints
Links:
- added link gripper_base_link; collision box size=0.03 0.025 0.03; visual box size=0.03 0.025 0.03
- added link left_gripper_finger_link; collision box size=0.015 0.01 0.01; collision box size=0.02 0.01 0.04
- added link right_gripper_finger_link; collision box size=0.015 0.01 0.01; collision box size=0.02 0.01 0.04
Joints:
- added joint gripper_base_joint: type fixed, parent wrist_tool_link, child gripper_base_link, origin xyz=0 0 0.02 rpy=0 0 0
- added joint gripper_joint: type prismatic, parent gripper_base_link, child left_gripper_finger_link, origin xyz=0 0.0125 0.03 rpy=0 0 0, axis 0 1 0, limit lower=-0.012 upper=0.012 effort=10 velocity=0.02
- added joint right_gripper_joint: type prismatic, parent gripper_base_link, child right_gripper_finger_link, origin xyz=0 -0.0125 0.03 rpy=0 0 0, axis 0 -1 0, limit lower=-0.012 upper=0.012 effort=10 velocity=0.02, mimic joint=gripper_joint multiplier=1.0 offset=0

File: r12_moveit_config/config/r12.ros2_control.xacro (robot description, xacro)
@@ -43,4 +43,11 @@
                 <state_interface name="velocity"/>
             </joint>
+            <joint name="gripper_joint">
+                <command_interface name="position"/>
+                <state_interface name="position">
+                  <param name="initial_value">${initial_positions['gripper_joint']}</param>
+                </state_interface>
+                <state_interface name="velocity"/>
+            </joint>
         </ros2_control>
     </xacro:macro>

Commit message: moveit2 and gz sim integration

File: r12_description/urdf/r12.urdf (robot description, URDF)
Before this commit: robot r12, 9 links, 8 joints
Links:
- link base_link: mass None -> 2.0
- link elbow_hand_link: mass None -> 0.6
- link gripper_base_link: mass None -> 0.1
- link hand_wrist_link: mass None -> 0.2
- link left_gripper_finger_link: mass None -> 0.05
- link right_gripper_finger_link: mass None -> 0.05
- link shoulder_elbow_link: mass None -> 1.2
- link waist_shoulder_link: mass None -> 0.8
- link wrist_tool_link: mass None -> 0.15

Commit message: urdf mimic joint fix

File: r12_description/urdf/r12.urdf (robot description, URDF)
Before this commit: robot r12, 9 links, 8 joints
Links:
- added link random
Joints:
- added joint right_gripper_joint_mimic: type fixed, parent base_link, child random
- joint elbow_joint: limit lower=-2.26 upper=2.26 effort=0.1 velocity=0.005 -> lower=-2.26 upper=2.26 effort=5.0 velocity=1.0
- joint hand_joint: limit lower=-2.09 upper=2.09 effort=0.1 velocity=0.005 -> lower=-2.09 upper=2.09 effort=5.0 velocity=1.0
- joint shoulder_joint: limit lower=-3.14159 upper=3.14159 effort=0.1 velocity=0.005 -> lower=-3.14159 upper=3.14159 effort=5.0 velocity=1.0
- joint waist_joint: limit lower=-3.14159 upper=3.14159 effort=0.1 velocity=0.005 -> lower=-3.14159 upper=3.14159 effort=5.0 velocity=1.0
- joint wrist_joint: limit lower=-3.14159 upper=3.14159 effort=0.1 velocity=0.005 -> lower=-3.14159 upper=3.14159 effort=5.0 velocity=1.0

Commit message: add realsense d435

File: r12_description/urdf/r12.urdf (robot description, URDF)
Before this commit: robot r12, 10 links, 9 joints
Links:
- added link rgbd_camera_frame, mass 0.072; collision box size=0.090 0.025 0.025; visual mesh filename=$(find depth_d435)/meshes/d435.dae scale=1.0 1.0 1.0
Joints:
- added joint rgbd_camera_joint: type fixed, parent base_link, child rgbd_camera_frame, origin xyz=0 0 1.0 rpy=0 0.5 0

Commit message: add perceprion

File: r12_description/urdf/r12.urdf (robot description, URDF)
Before this commit: robot r12, 11 links, 10 joints
Joints:
- joint rgbd_camera_joint: origin xyz=0 0 1.0 rpy=0 0.5 0 -> xyz=0.2 0 1.0 rpy=0 1.4 0
